Commit message: Added fake controller initial state

File: config/panda_arm_hand.srdf.xacro (robot description, xacro)
@@ -12,5 +12,6 @@
   <xacro:include filename="$(find panda_moveit_config)/config/hand.xacro" />
   <xacro:panda_arm />
-  <xacro:hand gripper_center="${gripper_center}" /> <!-- Added extra xacro macro argument for the new virtual center gripper link -->
+  <xacro:hand gripper_center="${gripper_center}" />
+  <!-- Added extra xacro macro argument for the new virtual center gripper link -->
   <!--GROUPS: Representation of a set of joints and links. This can be useful for specifying DOF to plan for, defining arms, end effectors, etc-->
   <!--LINKS: When a link is specified, the parent joint of that link (if it exists) is automatically included-->
@@ -42,6 +43,6 @@
   </group_state>
   <group_state name="open" group="hand">
-    <joint name="panda_finger_joint1" value="0.035" />
-    <joint name="panda_finger_joint2" value="0.035" />
+    <joint name="panda_finger_joint1" value="0.04" />
+    <joint name="panda_finger_joint2" value="0.04" />
   </group_state>
   <group_state name="close" group="hand">
@@ -52,6 +53,7 @@
   <end_effector name="hand" parent_link="panda_link8" group="hand" parent_group="panda_arm" />
   <!-- Added extra virtual joint to ease the grasp movement planning -->
-  <xacro:if value="${gripper_center}"> <!-- Only when gripper_center==True -->
+  <xacro:if value="${gripper_center}">    <!-- Only when gripper_center==True -->
     <end_effector name="gripper_center" parent_link="panda_gripper_center" group="panda_arm" parent_group="hand" />
+    <end_effector name="gripper_center" parent_link="panda_gripper_center" group="panda_arm_hand" />
   </xacro:if>
   <!--DISABLE COLLISIONS: By default it is assumed that any link of the robot could potentially come into collision with any other link in the robot. This tag disables collision checking between a specified pair of links. -->

Commit message: Changed gripper open named target

File: config/panda_arm_hand.srdf.xacro (robot description, xacro)
@@ -43,6 +43,7 @@
   </group_state>
   <group_state name="open" group="hand">
-    <joint name="panda_finger_joint1" value="0.04" />
-    <joint name="panda_finger_joint2" value="0.04" />
+    <!--Has to be set a little less than the maximum otherwise moveit won't plan -->
+    <joint name="panda_finger_joint1" value="0.035" />
+    <joint name="panda_finger_joint2" value="0.035" />
   </group_state>
   <group_state name="close" group="hand">
