Commit message: Added extra virtual gripper_center end effector to panda_arm_hand.srdf

File: config/hand.xacro (robot description, xacro)
@@ -11,4 +11,5 @@
       <link name="panda_leftfinger" />
       <link name="panda_rightfinger" />
+      <link name="panda_gripper_center" /> <!-- Added extra virutal joint to easy grasp movement planning -->
       <joint name="panda_finger_joint1" />
       <passive_joint name="panda_finger_joint2" />

File: config/panda_arm_hand.srdf.xacro (robot description, xacro)
@@ -47,4 +47,6 @@
   <!--END EFFECTOR: Purpose: Represent information about an end effector.-->
   <end_effector name="hand" parent_link="panda_link8" group="hand" parent_group="panda_arm" />
+  <!-- Added extra end effector to easy grasp movement planning -->
+  <end_effector name="gripper_center" parent_link="panda_gripper_center" group="panda_arm" parent_group="hand" />
   <!--DISABLE COLLISIONS: By default it is assumed that any link of the robot could potentially come into collision with any other link in the robot. This tag disables collision checking between a specified pair of links. -->
   <disable_collisions link1="panda_hand" link2="panda_link3" reason="Never" />

Commit message: Added extra virtual gripper_center end effector to panda_arm_hand.srdf
- Added virtual gripper to moveit groups

- Added virtual center gripper xacro:if statement

- Added gripper_center launch file arguments

File: config/hand.xacro (robot description, xacro)
@@ -1,5 +1,5 @@
 <?xml version="1.0" ?>
 <robot xmlns:xacro="http://www.ros.org/wiki/xacro" name="panda">
-  <xacro:macro name="hand">
+  <xacro:macro name="hand" params="gripper_center:='false'">
     <!--GROUPS: Representation of a set of joints and links. This can be useful for specifying DOF to plan for, defining arms, end effectors, etc-->
     <!--LINKS: When a link is specified, the parent joint of that link (if it exists) is automatically included-->
@@ -11,4 +11,8 @@
       <link name="panda_leftfinger" />
       <link name="panda_rightfinger" />
+      <!-- Added extra virtual joint to ease the grasp movement planning -->
+      <xacro:if value="${gripper_center}"> <!-- Only when gripper_center==True -->
+        <link name="panda_gripper_center" />
+      </xacro:if>
       <joint name="panda_finger_joint1" />
       <passive_joint name="panda_finger_joint2" />

File: config/panda_arm_hand.srdf.xacro (robot description, xacro)
@@ -5,8 +5,12 @@
 -->
 <robot xmlns:xacro="http://www.ros.org/wiki/xacro" name="panda">
+  <!-- Initialize gripper_center properties -->
+  <xacro:arg name="gripper_center" default="false" />
+  <xacro:property name="gripper_center" value="$(arg gripper_center)"/>
+  <!-- Include other subgroup xacros -->
   <xacro:include filename="$(find panda_moveit_config)/config/panda_arm.xacro" />
   <xacro:include filename="$(find panda_moveit_config)/config/hand.xacro" />
   <xacro:panda_arm />
-  <xacro:hand />
+  <xacro:hand gripper_center="${gripper_center}" /> <!-- Added extra xacro macro argument for the new virtual center gripper link -->
   <!--GROUPS: Representation of a set of joints and links. This can be useful for specifying DOF to plan for, defining arms, end effectors, etc-->
   <!--LINKS: When a link is specified, the parent joint of that link (if it exists) is automatically included-->
@@ -47,4 +51,8 @@
   <!--END EFFECTOR: Purpose: Represent information about an end effector.-->
   <end_effector name="hand" parent_link="panda_link8" group="hand" parent_group="panda_arm" />
+  <!-- Added extra virtual joint to ease the grasp movement planning -->
+  <xacro:if value="${gripper_center}"> <!-- Only when gripper_center==True -->
+    <end_effector name="gripper_center" parent_link="panda_gripper_center" group="panda_arm" parent_group="hand" />
+  </xacro:if>
   <!--DISABLE COLLISIONS: By default it is assumed that any link of the robot could potentially come into collision with any other link in the robot. This tag disables collision checking between a specified pair of links. -->
   <disable_collisions link1="panda_hand" link2="panda_link3" reason="Never" />

Commit message: :sparkles: Adds virtual grip site link
In order to control the robot w.r.t. the center of the gripper a virtual grip site link and joint were added.

File: config/hand.xacro (robot description, xacro)
@@ -1,5 +1,5 @@
 <?xml version="1.0" ?>
 <robot xmlns:xacro="http://www.ros.org/wiki/xacro" name="panda">
-  <xacro:macro name="hand">
+  <xacro:macro name="hand" params="grip_site:='false'">
     <!--GROUPS: Representation of a set of joints and links. This can be useful for specifying DOF to plan for, defining arms, end effectors, etc-->
     <!--LINKS: When a link is specified, the parent joint of that link (if it exists) is automatically included-->
@@ -11,4 +11,9 @@
       <link name="panda_leftfinger" />
       <link name="panda_rightfinger" />
+      <!-- Add extra virtual grip site joint -->
+      <xacro:if value="${grip_site}">
+        <!-- Only when grip_site==True -->
+        <link name="panda_grip_site" />
+      </xacro:if>
       <joint name="panda_finger_joint1" />
       <passive_joint name="panda_finger_joint2" />

File: config/panda_arm_hand.srdf.xacro (robot description, xacro)
@@ -7,6 +7,9 @@
   <xacro:include filename="$(find panda_moveit_config)/config/panda_arm.xacro" />
   <xacro:include filename="$(find panda_moveit_config)/config/hand.xacro" />
+  <!-- Initialize grip_site properties -->
+  <xacro:arg name="grip_site" default="false" />
+  <xacro:property name="grip_site" value="$(arg grip_site)" />
   <xacro:panda_arm />
-  <xacro:hand />
+  <xacro:hand grip_site="${grip_site}" />
   <!--GROUPS: Representation of a set of joints and links. This can be useful for specifying DOF to plan for, defining arms, end effectors, etc-->
   <!--LINKS: When a link is specified, the parent joint of that link (if it exists) is automatically included-->
@@ -27,5 +30,13 @@
   </group_state>
   <!--END EFFECTOR: Purpose: Represent information about an end effector.-->
-  <end_effector name="hand" parent_link="panda_link8" group="hand" parent_group="panda_arm" />
+  <xacro:unless value="${grip_site}">
+    <end_effector name="hand" parent_link="panda_link8" group="hand" parent_group="panda_arm" />
+  </xacro:unless>
+  <!-- Added virtual grip site joint -->
+  <xacro:if value="${grip_site}">
+    <!-- Only when grip_site==True -->
+    <end_effector name="grip_site" parent_link="panda_grip_site" group="panda_arm" parent_group="hand" />
+    <end_effector name="grip_site" parent_link="panda_grip_site" group="panda_arm_hand" />
+  </xacro:if>
   <!--DISABLE COLLISIONS: By default it is assumed that any link of the robot could potentially come into collision with any other link in the robot. This tag disables collision checking between a specified pair of links. -->
   <disable_collisions link1="panda_hand" link2="panda_link3" reason="Never" />
